File: toshiba-64mbit-adapter.sch (KiCad schematic (older format))
At the start: 9 parts, among them U1 TC5364205, U2 W29GL064C, U3 74HCT244, U4 74HCT244, U5 74HCT244, U6 74HCT244, U7 74HCT244, U8 TPS73633DBV

Commit message: v1.1
Connections:
- net A21: now also U1.11 (/E); no longer U1.13 (A21)
- net E: now also U1.13 (A21); no longer U1.11 (/E)
Changed lines of the file:
@@
 Text Label 2900 2400 2    50   ~ 10
 A0
-Text Label 2900 2500 2    50   ~ 10
+Text Label 2900 2700 2    50   ~ 10
 E
 Text Label 2900 2800 2    50   ~ 10
@@
 	1    0    0    -1
 $EndComp
-Text Label 2900 2700 2    50   ~ 0
+Text Label 2900 2500 2    50   ~ 0
 A21
 $Comp

Commit message: Change HCT to LVC chips to reflect constructed version.
Parts:
- U3, U4, U5, U6, U7: value 74HCT244 -> 74LVC244; symbol 74xx:74HCT244 -> toshiba-64mbit-adapter-rescue:74HCT244-74xx
Changed lines of the file:
@@
 EESchema Schematic File Version 4
-LIBS:toshiba-64mbit-adapter-cache
-EELAYER 29 0
+EELAYER 30 0
 EELAYER END
 $Descr A4 11693 8268
@@
 	2650 2600 2900 2600
 $Comp
-L 74xx:74HCT244 U4
+L toshiba-64mbit-adapter-rescue:74HCT244-74xx U4
 U 1 1 5C861A2E
 P 6350 3350
 F 0 "U4" H 6350 4331 50  0000 C CNN
-F 1 "74HCT244" H 6350 4240 50  0000 C CNN
+F 1 "74LVC244" H 6350 4240 50  0000 C CNN
 F 2 "Package_SO:TSSOP-20_4.4x6.5mm_P0.65mm" H 6350 3350 50  0001 C CNN
 F 3 "https://assets.nexperia.com/documents/data-sheet/74HC_HCT244.pdf" H 6350 3350 50  0001 C CNN
@@
 $EndComp
 $Comp
-L 74xx:74HCT244 U5
+L toshiba-64mbit-adapter-rescue:74HCT244-74xx U5
 U 1 1 5C8634EA
 P 7950 3350
 F 0 "U5" H 7950 4331 50  0000 C CNN
-F 1 "74HCT244" H 7950 4240 50  0000 C CNN
+F 1 "74LVC244" H 7950 4240 50  0000 C CNN
 F 2 "Package_SO:TSSOP-20_4.4x6.5mm_P0.65mm" H 7950 3350 50  0001 C CNN
 F 3 "https://assets.nexperia.com/documents/data-sheet/74HC_HCT244.pdf" H 7950 3350 50  0001 C CNN
@@
 $EndComp
 $Comp
-L 74xx:74HCT244 U7
+L toshiba-64mbit-adapter-rescue:74HCT244-74xx U7
 U 1 1 5C863DE8
 P 9400 3350
 F 0 "U7" H 9400 4331 50  0000 C CNN
-F 1 "74HCT244" H 9400 4240 50  0000 C CNN
+F 1 "74LVC244" H 9400 4240 50  0000 C CNN
 F 2 "Package_SO:TSSOP-20_4.4x6.5mm_P0.65mm" H 9400 3350 50  0001 C CNN
 F 3 "https://assets.nexperia.com/documents/data-sheet/74HC_HCT244.pdf" H 9400 3350 50  0001 C CNN
@@
 $EndComp
 $Comp
-L 74xx:74HCT244 U3
+L toshiba-64mbit-adapter-rescue:74HCT244-74xx U3
 U 1 1 5C865388
 P 6300 5450
 F 0 "U3" H 6300 6431 50  0000 C CNN
-F 1 "74HCT244" H 6300 6340 50  0000 C CNN
+F 1 "74LVC244" H 6300 6340 50  0000 C CNN
 F 2 "Package_SO:TSSOP-20_4.4x6.5mm_P0.65mm" H 6300 5450 50  0001 C CNN
 F 3 "https://assets.nexperia.com/documents/data-sheet/74HC_HCT244.pdf" H 6300 5450 50  0001 C CNN
@@
 $EndComp
 $Comp
-L 74xx:74HCT244 U6
+L toshiba-64mbit-adapter-rescue:74HCT244-74xx U6
 U 1 1 5C865EC6
 P 8000 5400
 F 0 "U6" H 8000 6381 50  0000 C CNN
-F 1 "74HCT244" H 8000 6290 50  0000 C CNN
+F 1 "74LVC244" H 8000 6290 50  0000 C CNN
 F 2 "Package_SO:TSSOP-20_4.4x6.5mm_P0.65mm" H 8000 5400 50  0001 C CNN
 F 3 "https://assets.nexperia.com/documents/data-sheet/74HC_HCT244.pdf" H 8000 5400 50  0001 C CNN
